Commit message: 改墙1碰撞半径

File: walls/wall1/wall2_1.urdf (robot description, URDF)
Before this commit: robot wall2_1.urdf, 1 links, 0 joints
Links:
- link baseLink: geometry collision box size=0.1 0.06 0.01; visual mesh filename=wall2_1.obj scale=1.0 1.0 1.0

Commit message: 做尝试

File: walls/wall1/wall2_1.urdf (robot description, URDF)
Before this commit: robot wall2_1.urdf, 1 links, 0 joints
Links:
- link baseLink: geometry collision mesh filename=wall2_1.obj scale=1.0 1.0 1.0; visual mesh filename=wall2_1.obj scale=1.0 1.0 1.0
